Commit message: the sim camera now works in rviz

File: moonpie_osamu/urdf/robot.urdf (robot description, URDF)
Before this commit: robot four_wheeled_robot, 6 links, 5 joints
Links:
- added link camera1_depth_optical_frame, mass 0.05; collision box size=0.03 0.03 0.03; visual box size=0.03 0.03 0.03
- added link camera1_link, mass 0.1; collision box size=0.05 0.05 0.05; visual box size=0.05 0.05 0.05
Joints:
- added joint camera1_joint: type fixed, parent base_link, child camera1_link, origin xyz=0.2 0 0.05 rpy=0 0 0
- added joint camera1_optical_joint: type fixed, parent camera1_link, child camera1_depth_optical_frame, origin xyz=0 0 0 rpy=0 0 0
- joint front_left_wheel_joint: origin xyz=0.2 0.15 0.05 rpy=1.5708 0 0 -> xyz=0.2 0.15 -0.05 rpy=1.5708 0 0
- joint front_right_wheel_joint: origin xyz=0.2 -0.15 0.05 rpy=1.5708 0 0 -> xyz=0.2 -0.15 -0.05 rpy=1.5708 0 0
- joint rear_left_wheel_joint: origin xyz=-0.2 0.15 0.05 rpy=1.5708 0 0 -> xyz=-0.2 0.15 -0.05 rpy=1.5708 0 0
- joint rear_right_wheel_joint: origin xyz=-0.2 -0.15 0.05 rpy=1.5708 0 0 -> xyz=-0.2 -0.15 -0.05 rpy=1.5708 0 0

Commit message: fixed some lingering issues

File: moonpie_osamu/urdf/robot.urdf (robot description, URDF)
Before this commit: robot four_wheeled_robot, 8 links, 7 joints
Links:
- removed link camera1_depth_optical_frame
Joints:
- removed joint camera1_optical_joint

Commit message: fixed some transforms; robot shows up right

File: moonpie_osamu/urdf/robot.urdf (robot description, URDF)
Before this commit: robot four_wheeled_robot, 7 links, 6 joints
Links:
- removed link world
- added link odom
Joints:
- removed joint world_to_base
- added joint odom_to_base: type fixed, parent odom, child base_link, origin xyz=0 0 0 rpy=0 0 0

Commit message: modified robot display to better match robot dimensions

File: moonpie_osamu/urdf/robot.urdf (robot description, URDF)
Before this commit: robot four_wheeled_robot, 7 links, 6 joints
Links:
- link base_link: geometry collision box size=1.1 0.7 0.35; visual box size=1.1 0.7 0.35
- link front_left_wheel: geometry collision cylinder length=0.1 radius=0.15; visual cylinder length=0.1 radius=0.15
- link front_right_wheel: geometry collision cylinder length=0.1 radius=0.15; visual cylinder length=0.1 radius=0.15
- link rear_left_wheel: geometry collision cylinder length=0.1 radius=0.15; visual cylinder length=0.1 radius=0.15
- link rear_right_wheel: geometry collision cylinder length=0.1 radius=0.15; visual cylinder length=0.1 radius=0.15
Joints:
- joint camera1_joint: origin xyz=0.2 0 0.05 rpy=0 0 0 -> xyz=0.55 0 0.32 rpy=0 0 0
- joint front_left_wheel_joint: origin xyz=0.2 0.15 -0.05 rpy=1.5708 0 0 -> xyz=0.5 0.3 0.15 rpy=1.5708 0 0
- joint front_right_wheel_joint: origin xyz=0.2 -0.15 -0.05 rpy=1.5708 0 0 -> xyz=0.5 -0.3 0.15 rpy=1.5708 0 0
- joint rear_left_wheel_joint: origin xyz=-0.2 0.15 -0.05 rpy=1.5708 0 0 -> xyz=-0.5 0.3 0.15 rpy=1.5708 0 0
- joint rear_right_wheel_joint: origin xyz=-0.2 -0.15 -0.05 rpy=1.5708 0 0 -> xyz=-0.5 -0.3 0.15 rpy=1.5708 0 0

Commit message: make a thingy

File: moonpie_osamu/urdf/robot.urdf (robot description, URDF)
Before this commit: robot four_wheeled_robot, 7 links, 6 joints
Links:
- added link dump_link, mass 0.1; collision box size=0.05 0.05 0.05; visual box size=0.05 0.05 0.05
Joints:
- added joint dump_joint: type fixed, parent base_link, child dump_link, origin xyz=-0.55 0 0.32 rpy=0 0 0
